Commit message: Added Camera sesnor to urdf added new world file with sensor plugins added world folder to cmakelist updated launch file to launch with new world

File: src/giraffe_description/urdf/giraffe.urdf.xacro (robot description, xacro)
@@ -148,4 +148,31 @@
         </collision>
     </link>
+    <link name="wrist_camera_link">
+        <inertial>
+            <origin xyz="0 0 0" rpy="0 0 0"/>
+            <mass value="0.03"/>
+            <inertia ixx="0.00001" iyy="0.00001" izz="0.00001"
+                    ixy="0" ixz="0" iyz="0"/>
+        </inertial>
+        <visual>
+            <origin xyz="0 0 0" rpy="0 0 0"/>
+            <geometry>
+                <box size="0.005 0.035 0.025"/>
+            </geometry>
+            <material name="blue"/>
+        </visual>
+        <collision>
+            <origin xyz="0 0 0" rpy="0 0 0"/>
+            <geometry>
+                <box size="0.005 0.035 0.025"/>
+            </geometry>
+        </collision>
+    </link>
+    <joint name="wrist_2_wrist_camera_joint" type="fixed">
+        <parent link="wrist_2"/>
+        <child link="wrist_camera_link"/>
+        <!-- Tune xyz/rpy after seeing it in RViz/Gazebo -->
+        <origin xyz="0.0 0 -0.03725" rpy="0 0 0"/>
+    </joint>
     <joint name="world_joint" type="fixed">
         <parent link="world" />
@@ -255,3 +282,24 @@
         </actuator>
     </transmission>
+    <gazebo reference="wrist_camera_link">
+        <sensor name="wrist_camera" type="camera">
+            <pose>0 0 0 0 0 0</pose>
+            <always_on>true</always_on>
+            <visualize>true</visualize>
+            <update_rate>30</update_rate>
+            <topic>/wrist_camera/image</topic>
+            <camera>
+                <horizontal_fov>1.047</horizontal_fov>
+                <image>
+                    <width>640</width>
+                    <height>480</height>
+                    <format>R8G8B8</format>
+                </image>
+                <clip>
+                    <near>0.02</near>
+                    <far>10.0</far>
+                </clip>
+            </camera>
+        </sensor>
+    </gazebo>
 </robot>

Commit message: Fixed Camera Position

File: src/giraffe_description/urdf/giraffe.urdf.xacro (robot description, xacro)
@@ -158,5 +158,5 @@
             <origin xyz="0 0 0" rpy="0 0 0"/>
             <geometry>
-                <box size="0.005 0.035 0.025"/>
+                <box size="0.005 0.035 0.0275"/>
             </geometry>
             <material name="blue"/>
@@ -165,5 +165,5 @@
             <origin xyz="0 0 0" rpy="0 0 0"/>
             <geometry>
-                <box size="0.005 0.035 0.025"/>
+                <box size="0.005 0.035 0.0275"/>
             </geometry>
         </collision>
@@ -173,5 +173,5 @@
         <child link="wrist_camera_link"/>
         <!-- Tune xyz/rpy after seeing it in RViz/Gazebo -->
-        <origin xyz="0.0 0 -0.03725" rpy="0 0 0"/>
+        <origin xyz="0.001 0 -0.0385" rpy="0 0 0"/>
     </joint>
     <joint name="world_joint" type="fixed">
@@ -284,5 +284,5 @@
     <gazebo reference="wrist_camera_link">
         <sensor name="wrist_camera" type="camera">
-            <pose>0 0 0 0 0 0</pose>
+            <pose>0 0 -0.006 3.14 0 3.14</pose>
             <always_on>true</always_on>
             <visualize>true</visualize>

Commit message: Added then commented out overhead camera

File: src/giraffe_description/urdf/giraffe.urdf.xacro (robot description, xacro)
@@ -303,3 +303,50 @@
         </sensor>
     </gazebo>
+    <!-- <link name="overhead_camera_link">
+        <inertial>
+            <origin xyz="0 0 0" rpy="0 0 0"/>
+            <mass value="0.03"/>
+            <inertia ixx="0.00001" iyy="0.00001" izz="0.00001"
+                    ixy="0" ixz="0" iyz="0"/>
+        </inertial>
+        <visual>
+            <origin xyz="0.00 -0.25 0.0" rpy="0 0.785  0"/>
+            <geometry>
+                <box size="0.005 0.5 0.0275"/>
+            </geometry>
+            <material name="blue"/>
+        </visual>
+        <collision>
+            <origin xyz="0.00 -0.25 0.0" rpy="0 0.785  0"/>
+            <geometry>
+                <box size="0.005 0.5 0.0275"/>
+            </geometry>
+        </collision>
+    </link>
+    <joint name="overhead_camera_joint" type="fixed">
+        <parent link="world"/>
+        <child link="overhead_camera_link"/>
+        <origin xyz="0.3 0.0 0" rpy="-1.57 0 0"/>
+    </joint>
+    <gazebo reference="overhead_camera_link">
+        <sensor name="overhead_camera" type="rgbd_camera">
+            <pose>0.0 -0.25 0 1.57 3.925 -0.3925</pose>
+            <always_on>true</always_on>
+            <visualize>true</visualize>
+            <update_rate>30</update_rate>
+            <topic>overhead_camera</topic>
+            <camera>
+                <horizontal_fov>1.047</horizontal_fov>
+                <image>
+                    <width>320</width>
+                    <height>240</height>
+                    <format>R8G8B8</format>
+                </image>
+                <clip>
+                    <near>0.05</near>
+                    <far>5.0</far>
+                </clip>
+            </camera>
+        </sensor>
+    </gazebo> -->
 </robot>

Commit message: Fixed Position and Added working Overhead camera

File: src/giraffe_description/urdf/giraffe.urdf.xacro (robot description, xacro)
@@ -303,5 +303,5 @@
         </sensor>
     </gazebo>
-    <!-- <link name="overhead_camera_link">
+    <link name="overhead_camera_link">
         <inertial>
             <origin xyz="0 0 0" rpy="0 0 0"/>
@@ -325,7 +325,7 @@
     </link>
     <joint name="overhead_camera_joint" type="fixed">
-        <parent link="world"/>
+        <parent link="base_link"/>
         <child link="overhead_camera_link"/>
-        <origin xyz="0.3 0.0 0" rpy="-1.57 0 0"/>
+        <origin xyz="-0.15 -0.2 0" rpy="-1.57 0 -1.57"/>
     </joint>
     <gazebo reference="overhead_camera_link">
@@ -349,4 +349,4 @@
             </camera>
         </sensor>
-    </gazebo> -->
+    </gazebo>
 </robot>

Commit message: Removed Wrist camera cause it was causing issue with moveit code and Removing Clutter from git status

File: src/giraffe_description/urdf/giraffe.urdf.xacro (robot description, xacro)
@@ -148,5 +148,5 @@
         </collision>
     </link>
-    <link name="wrist_camera_link">
+    <!-- <link name="wrist_camera_link">
         <inertial>
             <origin xyz="0 0 0" rpy="0 0 0"/>
@@ -168,11 +168,10 @@
             </geometry>
         </collision>
-    </link>
-    <joint name="wrist_2_wrist_camera_joint" type="fixed">
+    </link> -->
+    <!-- <joint name="wrist_2_wrist_camera_joint" type="fixed">
         <parent link="wrist_2"/>
         <child link="wrist_camera_link"/>
-        <!-- Tune xyz/rpy after seeing it in RViz/Gazebo -->
         <origin xyz="0.001 0 -0.0385" rpy="0 0 0"/>
-    </joint>
+    </joint> -->
     <joint name="world_joint" type="fixed">
         <parent link="world" />
@@ -282,5 +281,5 @@
         </actuator>
     </transmission>
-    <gazebo reference="wrist_camera_link">
+    <!-- <gazebo reference="wrist_camera_link">
         <sensor name="wrist_camera" type="rgbd_camera">
             <pose>0 0 -0.006 3.14 0 3.14</pose>
@@ -302,5 +301,5 @@
             </camera>
         </sensor>
-    </gazebo>
+    </gazebo> -->
     <link name="overhead_camera_link">
         <inertial>

Commit message: Added front camera and fixed position of front and overhead camera

File: src/giraffe_description/urdf/giraffe.urdf.xacro (robot description, xacro)
@@ -281,4 +281,30 @@
         </actuator>
     </transmission>
+    <!-- <link name="wrist_camera_link">
+        <inertial>
+            <origin xyz="0 0 0" rpy="0 0 0"/>
+            <mass value="0.03"/>
+            <inertia ixx="0.00001" iyy="0.00001" izz="0.00001"
+                    ixy="0" ixz="0" iyz="0"/>
+        </inertial>
+        <visual>
+            <origin xyz="0 0 0" rpy="0 0 0"/>
+            <geometry>
+                <box size="0.005 0.035 0.0275"/>
+            </geometry>
+            <material name="blue"/>
+        </visual>
+        <collision>
+            <origin xyz="0 0 0" rpy="0 0 0"/>
+            <geometry>
+                <box size="0.005 0.035 0.0275"/>
+            </geometry>
+        </collision>
+    </link> -->
+    <!-- <joint name="wrist_2_wrist_camera_joint" type="fixed">
+        <parent link="wrist_2"/>
+        <child link="wrist_camera_link"/>
+        <origin xyz="0.001 0 -0.0385" rpy="0 0 0"/>
+    </joint> -->
     <!-- <gazebo reference="wrist_camera_link">
         <sensor name="wrist_camera" type="rgbd_camera">
@@ -309,26 +335,26 @@
                     ixy="0" ixz="0" iyz="0"/>
         </inertial>
-        <visual>
-            <origin xyz="0.00 -0.25 0.0" rpy="0 0.785  0"/>
-            <geometry>
-                <box size="0.005 0.5 0.0275"/>
+        <!-- <visual>
+            <origin xyz="0.00 -0.0025 0.0" rpy="0 0 0"/>
+            <geometry>
+                <box size="0.005 0.005 0.005"/>
             </geometry>
             <material name="blue"/>
         </visual>
         <collision>
-            <origin xyz="0.00 -0.25 0.0" rpy="0 0.785  0"/>
-            <geometry>
-                <box size="0.005 0.5 0.0275"/>
-            </geometry>
-        </collision>
+            <origin xyz="0.00 -0.0025 0.0" rpy="0 0 0"/>
+            <geometry>
+                <box size="0.005 0.005 0.005"/>
+            </geometry>
+        </collision> -->
     </link>
     <joint name="overhead_camera_joint" type="fixed">
         <parent link="base_link"/>
         <child link="overhead_camera_link"/>
-        <origin xyz="-0.15 -0.2 0" rpy="-1.57 0 -1.57"/>
+        <origin xyz="0.25 -0.0 0.75" rpy="0 0 0"/>
     </joint>
     <gazebo reference="overhead_camera_link">
         <sensor name="overhead_camera" type="rgbd_camera">
-            <pose>0.0 -0.25 0 1.57 3.925 -0.3925</pose>
+            <pose>0 0 0 0 1.57 0</pose>
             <always_on>true</always_on>
             <visualize>true</visualize>
@@ -349,3 +375,37 @@
         </sensor>
     </gazebo>
+    <link name="front_camera_link">
+        <inertial>
+            <origin xyz="0 0 0" rpy="0 0 0"/>
+            <mass value="0.03"/>
+            <inertia ixx="0.00001" iyy="0.00001" izz="0.00001"
+                    ixy="0" ixz="0" iyz="0"/>
+        </inertial>
+    </link>
+    <joint name="front_camera_joint" type="fixed">
+        <parent link="base_link"/>
+        <child link="front_camera_link"/>
+        <origin xyz="1.0 -0.0 0" rpy="-1.57 0 3.14"/>
+    </joint>
+    <gazebo reference="front_camera_link">
+        <sensor name="front_camera" type="rgbd_camera">
+            <pose>0 -0.25 0 1.57 0 0</pose>
+            <always_on>true</always_on>
+            <visualize>true</visualize>
+            <update_rate>30</update_rate>
+            <topic>front_camera</topic>
+            <camera>
+                <horizontal_fov>1.047</horizontal_fov>
+                <image>
+                    <width>320</width>
+                    <height>240</height>
+                    <format>R8G8B8</format>
+                </image>
+                <clip>
+                    <near>0.05</near>
+                    <far>5.0</far>
+                </clip>
+            </camera>
+        </sensor>
+    </gazebo>
 </robot>

Commit message: Red Cube Detection Working correctly and Fixed orientation of overhead camera between joint and pose of camera and made relevant changes to tf in launch

File: src/giraffe_description/urdf/giraffe.urdf.xacro (robot description, xacro)
@@ -352,9 +352,9 @@
         <parent link="base_link"/>
         <child link="overhead_camera_link"/>
-        <origin xyz="0.25 -0.0 0.75" rpy="0 0 0"/>
+        <origin xyz="0.25 -0.0 0.75" rpy="0 1.57 0"/>
     </joint>
     <gazebo reference="overhead_camera_link">
         <sensor name="overhead_camera" type="rgbd_camera">
-            <pose>0 0 0 0 1.57 0</pose>
+            <pose>0 0 0 0 0 0</pose>
             <always_on>true</always_on>
             <visualize>true</visualize>
