Commit message: Fix gripper execution by updating URDF bounds/velocity limits, tuning Gazebo PID tolerances, and bypassing MTC execution with direct MoveGroupInterface trajectory execution

File: src/giraffe_description/urdf/giraffe.urdf.xacro (robot description, xacro)
@@ -219,5 +219,6 @@
         <child link="gripper" />
         <axis xyz="-0.007420635544791429 -0.0007590000001611277 -0.9999726580742655" />
-        <limit lower="0.0" upper="1.570796" effort="1000000" velocity="1000000" />
+        <!-- CHANGE THIS LINE -->
+        <limit lower="-0.05" upper="1.570796" effort="1000000" velocity="0.5" />
     </joint>
     <transmission name="shoulder_pan_trans">

Commit message: Pick and Place working

File: src/giraffe_description/urdf/giraffe.urdf.xacro (robot description, xacro)
@@ -220,5 +220,5 @@
         <axis xyz="-0.007420635544791429 -0.0007590000001611277 -0.9999726580742655" />
         <!-- CHANGE THIS LINE -->
-        <limit lower="-0.05" upper="1.570796" effort="1000000" velocity="0.5" />
+        <limit lower="-0.05" upper="1.570796" effort="1000000" velocity="1.0" />
     </joint>
     <transmission name="shoulder_pan_trans">

File: src/giraffe_description/urdf/giraffe_ros2_control.xacro (robot description, xacro)
@@ -2,5 +2,15 @@
 <robot name="giraffe" xmlns:xacro="http://www.ros.org/wiki/xacro" >
     <xacro:macro name="giraffe_ros2_control">
-            <gazebo>
+        <gazebo>
+            <!-- Add the Detachable Joint System -->
+            <!-- <plugin filename="gz-sim-detachable-joint-system"
+                    name="gz::sim::systems::DetachableJoint">
+                <parent_link>gripper</parent_link>
+                <child_model>red_cube</child_model>
+                <child_link>link</child_link>
+                <detach_topic>/detach_cube</detach_topic>
+                <attach_topic>/attach_cube</attach_topic>
+                <output_topic>/cube_state</output_topic>
+            </plugin> -->
             <plugin filename="ign_ros2_control-system" name="ign_ros2_control::IgnitionROS2ControlPlugin">
                 <robot_param>robot_description</robot_param>

Commit message: Added multiple cubes and cube and box detection to cube detector and fixed urdf colour

File: src/giraffe_description/urdf/giraffe.urdf.xacro (robot description, xacro)
@@ -7,5 +7,5 @@
     </material>
     <material name="white">
-        <color rgba="1 1 1 1"/>
+        <color rgba="0.68 0.70 0.73 1"/>
     </material>
     <link name="world"></link>
@@ -38,4 +38,5 @@
         <visual name="wrist_2_visual">
             <origin xyz="-0.021354214645274042 0.2206097855984012 -0.020899066496239235" rpy="-0.0008359974484128125 -1.562664271760666 3.135766541990315" />
+            <material name="white"/>
             <geometry>
                 <mesh filename="package://giraffe_description/meshes/wrist_2.stl" scale="0.001 0.001 0.001" />
@@ -57,5 +58,5 @@
         <visual name="wrist_1_visual">
             <origin xyz="0.02743385965284909 -0.010090686685202712 0.07569996720375094" rpy="-3.1415926535489875 0.0007586542251133366 1.2308559912525278e-10" />
-            <material name="blue"/>
+            <material name="white"/>
             <geometry>
                 <mesh filename="package://giraffe_description/meshes/wrist_1.stl" scale="0.001 0.001 0.001" />
@@ -97,4 +98,5 @@
         <visual name="shoulder_lift_visual">
             <origin xyz="0.013526461857575818 0.04663671319906652 0.1165941136588908" rpy="-1.5707963270017984 0.0007586542251355672 -2.0674688021030666e-10" />
+            <material name="white"/>
             <geometry>
                 <mesh filename="package://giraffe_description/meshes/shoulder_lift.stl" scale="0.001 0.001 0.001" />
@@ -116,5 +118,5 @@
         <visual name="shoulder_pan_visual">
             <origin xyz="-0.09115887303880836 0.0059308387053767 0.06458670903944891" rpy="-1.998138486507446e-15 1.56795957134278e-13 -1.570037672569761" />
-            <material name="blue"/>
+            <material name="white"/>
             <geometry>
                 <mesh filename="package://giraffe_description/meshes/shoulder_pan.stl" scale="0.001 0.001 0.001" />
@@ -160,5 +162,5 @@
                 <box size="0.005 0.035 0.0275"/>
             </geometry>
-            <material name="blue"/>
+            <material name="white"/>
         </visual>
         <collision>
@@ -294,5 +296,5 @@
                 <box size="0.005 0.035 0.0275"/>
             </geometry>
-            <material name="blue"/>
+            <material name="white"/>
         </visual>
         <collision>
@@ -341,5 +343,5 @@
                 <box size="0.005 0.005 0.005"/>
             </geometry>
-            <material name="blue"/>
+            <material name="white"/>
         </visual>
         <collision>

Commit message: Updated Readme, New media files, Removed text from cv window, Increased execution speed, fine tuned offsets in mtc code

File: src/giraffe_description/urdf/giraffe.urdf.xacro (robot description, xacro)
@@ -3,10 +3,13 @@
     <xacro:include filename="$(find giraffe_description)/urdf/giraffe_ros2_control.xacro" />
     <xacro:giraffe_ros2_control />
-    <material name="blue">
-        <color rgba="0 0 0.8 1"/>
+    <material name="color_1">
+        <color rgba="0.46 0.49 0.52 1"/>
     </material>
-    <material name="white">
+    <material name="color_2">
+        <color rgba="0.38 0.44 0.51 1"/>
+    </material>
+    <!-- <material name="white">
         <color rgba="0.68 0.70 0.73 1"/>
-    </material>
+    </material> -->
     <link name="world"></link>
     <link name="gripper">
@@ -18,5 +21,5 @@
         <visual name="gripper_visual">
             <origin xyz="-0.0033119954003824857 0.031004368928997047 0.2854674914428595" rpy="-1.578235904251224 0.0005414131158789297 -1.3962152952062392" />
-            <material name="white"/>
+            <material name="color_2"/>
             <geometry>
                 <mesh filename="package://giraffe_description/meshes/gripper.stl" scale="0.001 0.001 0.001" />
@@ -38,5 +41,5 @@
         <visual name="wrist_2_visual">
             <origin xyz="-0.021354214645274042 0.2206097855984012 -0.020899066496239235" rpy="-0.0008359974484128125 -1.562664271760666 3.135766541990315" />
-            <material name="white"/>
+            <material name="color_2"/>
             <geometry>
                 <mesh filename="package://giraffe_description/meshes/wrist_2.stl" scale="0.001 0.001 0.001" />
@@ -58,5 +61,5 @@
         <visual name="wrist_1_visual">
             <origin xyz="0.02743385965284909 -0.010090686685202712 0.07569996720375094" rpy="-3.1415926535489875 0.0007586542251133366 1.2308559912525278e-10" />
-            <material name="white"/>
+            <material name="color_1"/>
             <geometry>
                 <mesh filename="package://giraffe_description/meshes/wrist_1.stl" scale="0.001 0.001 0.001" />
@@ -78,5 +81,5 @@
         <visual name="elbow_visual">
             <origin xyz="-0.01857530598299039 0.008291687482204822 0.009868027761990259" rpy="-1.5707963267127854 -6.404382232928635e-16 3.1415926534651977" />
-            <material name="white"/>
+            <material name="color_2"/>
             <geometry>
                 <mesh filename="package://giraffe_description/meshes/elbow.stl" scale="0.001 0.001 0.001" />
@@ -98,5 +101,5 @@
         <visual name="shoulder_lift_visual">
             <origin xyz="0.013526461857575818 0.04663671319906652 0.1165941136588908" rpy="-1.5707963270017984 0.0007586542251355672 -2.0674688021030666e-10" />
-            <material name="white"/>
+            <material name="color_1"/>
             <geometry>
                 <mesh filename="package://giraffe_description/meshes/shoulder_lift.stl" scale="0.001 0.001 0.001" />
@@ -118,5 +121,5 @@
         <visual name="shoulder_pan_visual">
             <origin xyz="-0.09115887303880836 0.0059308387053767 0.06458670903944891" rpy="-1.998138486507446e-15 1.56795957134278e-13 -1.570037672569761" />
-            <material name="white"/>
+            <material name="color_1"/>
             <geometry>
                 <mesh filename="package://giraffe_description/meshes/shoulder_pan.stl" scale="0.001 0.001 0.001" />
@@ -138,5 +141,5 @@
         <visual name="base_link_visual">
             <origin xyz="0.0 0.0 0.0" rpy="0.0 0.0 0.0" />
-            <material name="white"/>
+            <material name="color_1"/>
             <geometry>
                 <mesh filename="package://giraffe_description/meshes/base_link.stl" scale="0.001 0.001 0.001" />
